Commit message: Gazebo bringup, live force interaction, and plotting.

File: packages/zfc_bringup/urdf/stage.urdf.xacro (robot description, xacro)
@@ -3,5 +3,5 @@
   <!-- REVIEW DRAFT. Geometry, masses, travel and limits are illustrative.
        Installation calibration must be measured before physical configuration.
-       This file prepares Gazebo integration; it is not a simulation launch. -->
+       Gazebo uses known illustrative bounds, not measured hardware bounds. -->
   <xacro:arg name="backend" default="ethercat"/>
   <xacro:arg name="controllers_file" default="${xacro.abs_filename('../config/controllers.yaml')}"/>
@@ -9,9 +9,11 @@
   <xacro:arg name="hardware_calibration_file" default="${xacro.abs_filename('../config/hardware_calibration.yaml')}"/>
   <xacro:arg name="travel_m" default="0.50"/>
-  <xacro:arg name="velocity_limit_mps" default="0.10"/>
+  <!-- Fortress velocity servo requires headroom above the 0.1 m/s trajectory;
+       at the exact DART velocity limit its response can remain saturated. -->
+  <xacro:arg name="velocity_limit_mps" default="${0.2 if '$(arg backend)' == 'gazebo' else 0.1}"/>
   <xacro:arg name="effort_limit_n" default="100.0"/>
   <xacro:arg name="carriage_mass_kg" default="2.0"/>
   <xacro:arg name="tool_mass_kg" default="0.20"/>
-  <xacro:arg name="initial_position_m" default="0.25"/>
+  <xacro:arg name="initial_position_m" default="0.0"/>
   <xacro:arg name="diagnostic_mode" default="production"/>
   <xacro:property name="backend" value="$(arg backend)"/>
@@ -21,4 +23,5 @@
   <xacro:property name="carriage_mass" value="$(arg carriage_mass_kg)"/>
   <xacro:property name="tool_mass" value="$(arg tool_mass_kg)"/>
+  <xacro:property name="simulation_datum" value="${0.25 if backend == 'gazebo' else 0.0}"/>
   <material name="rail_black"><color rgba="0.12 0.13 0.14 1"/></material>
   <material name="aluminium"><color rgba="0.65 0.68 0.70 1"/></material>
@@ -57,12 +60,12 @@
     </visual>
   </link>
-  <!-- Gazebo q=0 is the model lower datum. Hardware q=0 is a stationary
+  <!-- Gazebo q=0 is the KNOWN 0.25 m mid-travel session reference. Hardware q=0 is a stationary
        session reference: physical TF/mechanical offset remains unknown.
        +q is upward once encoder polarity is verified. -->
   <joint name="carriage" type="prismatic">
     <parent link="base_link"/><child link="carriage_link"/>
-    <origin xyz="0.09 0 0.20"/>
+    <origin xyz="${0.14 if backend == 'gazebo' else 0.09} 0 ${0.20+simulation_datum}"/>
     <axis xyz="0 0 1"/>
-    <limit lower="0.0" upper="${travel}" effort="$(arg effort_limit_n)"
+    <limit lower="${-simulation_datum}" upper="${travel-simulation_datum}" effort="$(arg effort_limit_n)"
            velocity="$(arg velocity_limit_mps)"/>
     <dynamics damping="0.0" friction="0.0"/>
@@ -87,5 +90,5 @@
   <joint name="tool_mount" type="fixed">
     <parent link="load_cell_link"/><child link="tool_link"/>
-    <origin xyz="0 0 -0.055"/>
+    <origin xyz="0 0 ${-0.06 if backend == 'gazebo' else -0.055}"/>
   </joint>
   <link name="tool_link">
@@ -127,5 +130,5 @@
              Physical session-relative soft bounds are independent calibration. -->
         <xacro:if value="${backend == 'gazebo'}">
-          <param name="min">0.0</param><param name="max">${travel}</param>
+          <param name="min">${-simulation_datum}</param><param name="max">${travel-simulation_datum}</param>
         </xacro:if>
       </command_interface>
@@ -135,5 +138,7 @@
         </xacro:if>
       </state_interface>
-      <state_interface name="velocity"/>
+      <state_interface name="velocity">
+        <xacro:if value="${backend == 'gazebo'}"><param name="initial_value">0.0</param></xacro:if>
+      </state_interface>
       <!-- No effort state until motor torque -> joint force is verified. -->
     </joint>
@@ -157,4 +162,6 @@
       </sensor>
     </gazebo>
+    <!-- Keep the force target an actual downstream link, not a merged alias. -->
+    <gazebo reference="tool_mount"><preserveFixedJoint>true</preserveFixedJoint></gazebo>
     <gazebo>
       <plugin filename="gz_ros2_control-system" name="gz_ros2_control::GazeboSimROS2ControlPlugin">
